File: BMP_BasicClone/BMP_BasicClone.kicad_pcb (KiCad board)
At the start: 2 copper layers, 112 x 204.7 mm, 53 parts, among them J1 BARREL_JACK, Q1 MMBT3904, Q2 MMBT3904, Q3 MMBT3904, Q4 MMBT3904

Commit message: Board Description Update
Other:
- board text added: "Hammond 1590G"
Changed lines of the file:
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@@
     (links 85)
     (no_connects 0)
-    (area 31.928999 27.864999 161.365001 232.739001)
+    (area 31.928999 27.864999 154.707001 232.739001)
     (thickness 1.6)
-    (drawings 37)
+    (drawings 38)
     (tracks 391)
     (zones 0)
@@
     (pad_to_mask_clearance 0.2)
     (aux_axis_origin 0 0)
-    (visible_elements FFFCFF7F)
+    (visible_elements 7FFEFFFF)
     (pcbplotparams
       (layerselection 0x00030_80000001)
@@
     )
   )
+  (gr_text "Hammond 1590G\n" (at 125.095 120.142) (layer F.SilkS)
+    (effects (font (size 1.5 1.5) (thickness 0.3)))
+  )
   (gr_line (start 107.188 218.948) (end 107.188 224.028) (angle 90) (layer Edge.Cuts) (width 0.15))
   (gr_line (start 102.108 218.948) (end 107.188 218.948) (angle 90) (layer Edge.Cuts) (width 0.15))
@@
   (segment (start 130.556 146.854) (end 130.514 146.854) (width 0.25) (layer F.Cu) (net 6) (status 10))
   (segment (start 130.5325 146.8775) (end 130.556 146.854) (width 0.25) (layer F.Cu) (net 6) (status 30))
-  (segment (start 137.414 196.046) (end 137.414 195.707) (width 0.25) (layer F.Cu) (net 7) (status 400000))
+  (segment (start 137.414 196.046) (end 137.414 195.707) (width 0.25) (layer F.Cu) (net 7))
   (segment (start 137.414 195.707) (end 134.366 192.659) (width 0.25) (layer F.Cu) (net 7))
   (segment (start 134.366 174.498) (end 137.287 171.577) (width 0.25) (layer F.Cu) (net 7))

Commit message: updates
Parts:
- R1: value R -> 1k
- SW_EN1: footprint custom_sw:SW_3PDT_W18MM_L17.3MM_P5.3MM_D2MM -> custom_sw:SW_3PDT_W18MM_L17.3MM_P5.3MM_D2MM_SolderLugs
Routing:
- net /+9V: track 171.9 -> 170.2 mm
Changed lines of the file:
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@@
     (links 85)
     (no_connects 0)
-    (area 31.928999 27.864999 154.707001 232.739001)
+    (area 31.928999 27.864999 144.093001 232.739001)
     (thickness 1.6)
     (drawings 38)
-    (tracks 391)
+    (tracks 390)
     (zones 0)
     (modules 53)
@@
       (effects (font (size 1 1) (thickness 0.15)))
     )
-    (fp_text value R (at 0 1.25) (layer F.Fab)
+    (fp_text value 1k (at 0 1.25) (layer F.Fab)
       (effects (font (size 1 1) (thickness 0.15)))
     )
@@
     )
   )
-  (module custom_sw:SW_3PDT_W18MM_L17.3MM_P5.3MM_D2MM (layer F.Cu)
-    (at 123.444 214.884)
-    (fp_text reference SW_EN1 (at 0 11.176) (layer F.SilkS)
-      (effects (font (size 1 1) (thickness 0.15)))
-    )
-    (fp_text value SW_3PDT_on_on (at 0.254 14.478) (layer F.Fab)
-      (effects (font (size 1 1) (thickness 0.15)))
-    )
-    (fp_line (start -8.89 -8.509) (end 7.62 -8.509) (layer F.SilkS) (width 0.15))
-    (fp_line (start 7.62 -8.509) (end 8.89 -8.509) (layer F.SilkS) (width 0.15))
-    (fp_line (start 9.017 -8.89) (end 9.017 8.89) (layer F.SilkS) (width 0.15))
-    (fp_line (start 8.89 8.509) (end -8.89 8.509) (layer F.SilkS) (width 0.15))
-    (fp_line (start -9.017 8.89) (end -9.017 -8.89) (layer F.SilkS) (width 0.15))
-    (pad 1 thru_hole oval (at -5.5 -4.6) (size 3.5 3) (drill 1.5) (layers *.Cu *.Mask)
-      (net 35 "Net-(SW_EN1-Pad1)"))
-    (pad 4 thru_hole oval (at 0 -4.6) (size 3.5 3) (drill 1.5) (layers *.Cu *.Mask)
-      (net 36 "Net-(SW_EN1-Pad4)"))
-    (pad 7 thru_hole oval (at 5.5 -4.6) (size 3.5 3) (drill 1.5) (layers *.Cu *.Mask)
-      (net 35 "Net-(SW_EN1-Pad1)"))
-    (pad 2 thru_hole oval (at -5.5 0) (size 3.5 3) (drill 1.5) (layers *.Cu *.Mask)
-      (net 30 "Net-(J_OUT1-Pad1)"))
-    (pad 5 thru_hole oval (at 0 0) (size 3.5 3) (drill 1.5) (layers *.Cu *.Mask)
-      (net 24 /+9V))
-    (pad 8 thru_hole oval (at 5.5 0) (size 3.5 3) (drill 1.5) (layers *.Cu *.Mask)
-      (net 27 "Net-(J_IN1-Pad1)"))
-    (pad 3 thru_hole oval (at -5.5 4.6) (size 3.5 3) (drill 1.5) (layers *.Cu *.Mask)
-      (net 34 "Net-(R26-Pad2)"))
-    (pad 6 thru_hole oval (at 0 4.6) (size 3.5 3) (drill 1.5) (layers *.Cu *.Mask)
-      (net 22 "Net-(D5-Pad2)"))
-    (pad 9 thru_hole oval (at 5.5 4.6) (size 3.5 3) (drill 1.5) (layers *.Cu *.Mask)
-      (net 32 "Net-(R2-Pad2)"))
-  )
   (module Diodes_SMD:D_SOD-323_HandSoldering (layer F.Cu)
     (at 110.236 170.688)
@@
       (rotate (xyz 0 0 0))
     )
+  )
+  (module custom_sw:SW_3PDT_W18MM_L17.3MM_P5.3MM_D2MM_SolderLugs (layer F.Cu)
+    (at 123.444 214.884)
+    (fp_text reference SW_EN1 (at 0 11.176) (layer F.SilkS)
+      (effects (font (size 1 1) (thickness 0.15)))
+    )
+    (fp_text value SW_3PDT_on_on (at 0.254 14.478) (layer F.Fab)
+      (effects (font (size 1 1) (thickness 0.15)))
+    )
+    (fp_line (start -8.89 -8.509) (end 7.62 -8.509) (layer F.SilkS) (width 0.15))
+    (fp_line (start 7.62 -8.509) (end 8.89 -8.509) (layer F.SilkS) (width 0.15))
+    (fp_line (start 9.017 -8.89) (end 9.017 8.89) (layer F.SilkS) (width 0.15))
+    (fp_line (start 8.89 8.509) (end -8.89 8.509) (layer F.SilkS) (width 0.15))
+    (fp_line (start -9.017 8.89) (end -9.017 -8.89) (layer F.SilkS) (width 0.15))
+    (pad 1 thru_hole oval (at -5.5 -4.6) (size 4 3.5) (drill 2) (layers *.Cu *.Mask)
+      (net 35 "Net-(SW_EN1-Pad1)"))
+    (pad 4 thru_hole oval (at 0 -4.6) (size 4 3.5) (drill 2) (layers *.Cu *.Mask)
+      (net 36 "Net-(SW_EN1-Pad4)"))
+    (pad 7 thru_hole oval (at 5.5 -4.6) (size 4 3.5) (drill 2) (layers *.Cu *.Mask)
+      (net 35 "Net-(SW_EN1-Pad1)"))
+    (pad 2 thru_hole oval (at -5.5 0) (size 4 3.5) (drill 2) (layers *.Cu *.Mask)
+      (net 30 "Net-(J_OUT1-Pad1)"))
+    (pad 5 thru_hole oval (at 0 0) (size 4 3.5) (drill 2) (layers *.Cu *.Mask)
+      (net 24 /+9V))
+    (pad 8 thru_hole oval (at 5.5 0) (size 4 3.5) (drill 2) (layers *.Cu *.Mask)
+      (net 27 "Net-(J_IN1-Pad1)"))
+    (pad 3 thru_hole oval (at -5.5 4.6) (size 4 3.5) (drill 2) (layers *.Cu *.Mask)
+      (net 34 "Net-(R26-Pad2)"))
+    (pad 6 thru_hole oval (at 0 4.6) (size 4 3.5) (drill 2) (layers *.Cu *.Mask)
+      (net 22 "Net-(D5-Pad2)"))
+    (pad 9 thru_hole oval (at 5.5 4.6) (size 4 3.5) (drill 2) (layers *.Cu *.Mask)
+      (net 32 "Net-(R2-Pad2)"))
   )
   (gr_text "Hammond 1590G\n" (at 125.095 120.142) (layer F.SilkS)
@@
   (segment (start 129.54 134.894) (end 124.028 134.64) (width 0.25) (layer F.Cu) (net 23) (status 10))
   (segment (start 124.028 134.64) (end 122.428 136.24) (width 0.25) (layer F.Cu) (net 23))
-  (segment (start 132.08 216.916) (end 132.08 215.9) (width 0.25) (layer F.Cu) (net 24))
+  (segment (start 132.334 215.646) (end 130.81 217.17) (width 0.25) (layer F.Cu) (net 24))
+  (segment (start 123.444 214.884) (end 125.73 217.17) (width 0.25) (layer F.Cu) (net 24) (status 400000))
+  (segment (start 125.73 217.17) (end 130.81 217.17) (width 0.25) (layer F.Cu) (net 24))
+  (segment (start 123.444 214.884) (end 121.158 212.598) (width 0.25) (layer F.Cu) (net 24) (status 400000))
+  (segment (start 116.078 212.598) (end 115.824 212.344) (width 0.25) (layer F.Cu) (net 24))
+  (segment (start 121.158 212.598) (end 116.078 212.598) (width 0.25) (layer F.Cu) (net 24))
+  (segment (start 132.334 215.646) (end 134.62 213.36) (width 0.25) (layer F.Cu) (net 24))
   (segment (start 134.62 213.36) (end 134.62 198.062) (width 0.25) (layer F.Cu) (net 24) (status 20))
-  (segment (start 132.08 215.9) (end 134.62 213.36) (width 0.25) (layer F.Cu) (net 24))
   (segment (start 129.032 164.592) (end 129.032 167.582) (width 0.25) (layer F.Cu) (net 24))
   (segment (start 129.032 167.582) (end 128.974 167.64) (width 0.25) (layer F.Cu) (net 24))
@@
   (segment (start 113.284 159.004) (end 115.316 156.972) (width 0.25) (layer F.Cu) (net 24))
   (segment (start 112.268 183.896) (end 122.358727 183.896) (width 0.25) (layer F.Cu) (net 24))
-  (segment (start 123.444 214.884) (end 121.412 212.852) (width 0.25) (layer F.Cu) (net 24))
-  (segment (start 121.412 212.852) (end 116.332 212.852) (width 0.25) (layer F.Cu) (net 24))
-  (segment (start 116.332 212.852) (end 115.316 211.836) (width 0.25) (layer F.Cu) (net 24))
+  (segment (start 115.824 212.344) (end 115.316 211.836) (width 0.25) (layer F.Cu) (net 24))
   (segment (start 115.316 211.836) (end 115.316 208.788) (width 0.25) (layer F.Cu) (net 24))
   (segment (start 115.316 208.788) (end 117.856 206.248) (width 0.25) (layer F.Cu) (net 24))
@@
   (segment (start 129.598 143.256) (end 129.598 139.7) (width 0.25) (layer F.Cu) (net 24) (status 10))
   (segment (start 134.62 198.062) (end 134.62 198.247) (width 0.25) (layer F.Cu) (net 24) (status 30))
-  (segment (start 131.572 217.424) (end 124.587 217.424) (width 0.25) (layer F.Cu) (net 24))
-  (segment (start 132.08 216.916) (end 131.572 217.424) (width 0.25) (layer F.Cu) (net 24))
-  (segment (start 124.587 217.424) (end 123.444 216.281) (width 0.25) (layer F.Cu) (net 24))
-  (segment (start 123.444 216.281) (end 123.444 214.884) (width 0.25) (layer F.Cu) (net 24))
   (segment (start 130.683 186.69) (end 130.683 205.105) (width 0.25) (layer F.Cu) (net 27))
   (segment (start 130.683 205.105) (end 131.953 206.375) (width 0.25) (layer F.Cu) (net 27))

Commit message: update
Parts:
- removed R24, R25, R26: 100K, Potentiometers:Potentiometer_Bourns_PTV09A-1_Horizontal
- added J2: CONN_02X06, Pin_Headers:Pin_Header_Straight_2x06_Pitch2.54mm, F.Cu at (74.2, 132.0)
- added J3: CONN_02X06, Pin_Headers:Pin_Header_Straight_2x06_Pitch2.54mm, F.Cu at (156.2, 146.8)
- added SUSTAIN1: 100K, Potentiometers:Potentiometer_Bourns_PTV09A-1_Horizontal, F.Cu at (240.3, 156.2)
- added TONE1: 100K, Potentiometers:Potentiometer_Bourns_PTV09A-1_Horizontal, F.Cu at (254.0, 155.7)
- added VOLUME1: 100K, Potentiometers:Potentiometer_Bourns_PTV09A-1_Horizontal, F.Cu at (225.0, 156.2)
- C1, C10, C11, C12, C13, C2, C3, C4, C5, C6, C7, C8, C9: footprint Capacitors_SMD:C_0402_NoSilk -> Capacitors_SMD:C_0805
- D1, D2, D3, D4, D6: footprint Diodes_SMD:D_SOD-323_HandSoldering -> Diodes_SMD:D_SOD-523
- R1, R10, R11, R12, R13, R14, R15, R16, R17, R18, R19, R2, R20, R21, R22, R23, R3, R4, R5, R6, R7, R8, R9: footprint Resistors_SMD:R_0402_NoSilk -> Resistors_SMD:R_0805
- moved J_IN1 60.1 mm to (83.9, 147.4)
- moved R22 58.6 mm to (91.9, 171.7)
- moved R14 58.4 mm to (95.0, 170.7)
- moved Q4 55.7 mm to (92.7, 184.7)
- moved C2 55.7 mm to (85.9, 105.8)
- moved R9 55.7 mm to (86.6, 190.8)
- moved C4 55.7 mm to (89.4, 168.4)
- moved C1 55.7 mm to (87.6, 193.3)
- moved J1 55.7 mm to (74.4, 114.0)
- moved Q1 55.7 mm to (86.5, 111.5)
- moved R13 55.7 mm to (86.6, 169.4)
- moved R2 55.7 mm to (85.1, 193.3)
- moved R23 55.7 mm to (88.4, 124.8)
- moved R6 55.7 mm to (82.0, 111.5)
- moved R7 55.7 mm to (82.0, 115.1)
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Connections:
- net Net-(C8-Pad1) renamed /TONE_P1
- net Net-(C9-Pad1) renamed /TONE_P3
- C2 pad 2: Net-(C2-Pad2) -> /VOL_P1
- C3 pad 2: Net-(C3-Pad2) -> /TONE_P2
- C4 pad 1: Net-(C4-Pad1) -> /SUS_P3
- C5 pad 1: Net-(C5-Pad1) -> /SUS_P2
- R1 pad 1: /GND -> Net-(D5-Pad1)
- R1 pad 2: Net-(D5-Pad1) -> Net-(J3-Pad2)
- R23 pad 1: Net-(R23-Pad1) -> /SUS_P1
- SW_EN1 pad 3: Net-(R26-Pad2) -> /VOL_P2
- SW_EN1 pad 6: Net-(D5-Pad2) -> /LED_AN
Routing:
- net /GND: track 240.4 -> 85.4 mm, vias 6 -> 2
- net /+9V: track 170.2 -> 35.4 mm, vias 4 -> 0
- net Net-(D5-Pad2): track 76.4 -> 0.00 mm, vias 4 -> 0
- net Net-(R26-Pad2): track 71.2 -> 0.00 mm
- net /VOL_P2: track 0.00 -> 62.0 mm
- net Net-(C2-Pad2): track 44.8 -> 0.00 mm
- net Net-(C4-Pad1): track 42.9 -> 0.00 mm
- net Net-(J_IN1-Pad1): track 45.1 -> 4.38 mm
- net Net-(D5-Pad1): track 41.2 -> 0.51 mm, vias 4 -> 0
- net Net-(C10-Pad1): track 32.7 -> 0.49 mm
- net Net-(J_IN1-Pad2): track 0.00 -> 31.0 mm
- net Net-(C1-Pad1): track 25.1 -> 0.33 mm
- net Net-(C3-Pad2): track 19.4 -> 0.00 mm
- net /TONE_P1: track 16.8 -> 0.04 mm, vias 2 -> 0
- net (no net): track 0.00 -> 10.9 mm
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Other:
- board size 112 x 204.7 mm -> 155.2 x 217.4 mm

Commit message: board update
Parts:
- C10: value 560pF -> 4.7nF
- C11: value 560pF -> 10nF
- C12: value 560pF -> 100nF
- C13, C3, C5: value 100nF -> 1uF
- C2, C6: value 1uF -> 560pF
- C4, C7: value 1uF -> 100nF
- C8: value 10nF -> 1uF
- C9: value 4.7nF -> 560pF
- D1: value 1N914 -> D_Schottky
- D5: value LED -> 1N914; footprint LEDs:LED_D5.0mm -> Diodes_SMD:D_SOD-523
- D6: value D_Schottky -> LED; footprint Diodes_SMD:D_SOD-523 -> LEDs:LED_D5.0mm
- R1: value 1k -> 39K
- R10: value 150R -> 10K
- R11: value 15K -> 150R
- R13: value 10K -> 100K
- R14, R3: value 100K -> 470K
- R15: value 470K -> 15K
- R16: value 100K -> 150R
- R17: value 470K -> 39K
- R18: value 10K -> 22K
- R19: value 10K -> 430K
- R2, R8: value 39K -> 100K
- R21: value 150R -> 15K
- R22: value 120R -> 3K3
- R23: value 1K -> 1k
- R4: value 3K3 -> 10K
- R5: value 22K -> 120R
- R6: value 15K -> 1K
- R7: value 430K -> 10K
- moved D6 106.4 mm to (170.8, 166.0)
- moved R19 84.7 mm to (59.5, 116.4), turned to 180 degrees
- moved R17 80.6 mm to (63.4, 126.9)
- moved R21 79.9 mm to (59.8, 140.8), turned to 270 degrees
- moved C2 77.8 mm to (89.4, 183.5), turned to 0 degrees
- moved R4 75.9 mm to (85.8, 189.8), turned to 90 degrees
- moved R23 74.2 mm to (155.7, 156.1)
- moved C5 72.8 mm to (87.4, 164.3), turned to 180 degrees
- moved C12 71.0 mm to (71.0, 126.9), turned to 270 degrees
- moved R20 69.5 mm to (71.5, 118.3), turned to 90 degrees
- moved D5 67.7 mm to (88.4, 125.1), turned to 270 degrees
- moved R5 66.7 mm to (91.0, 174.7), turned to 270 degrees
- moved Q1 65.1 mm to (87.0, 176.6)
- moved R1 64.7 mm to (93.9, 185.1), turned to 270 degrees
- moved C13 61.6 mm to (62.7, 140.4), turned to 90 degrees
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Connections:
- C10 pad 1: Net-(C10-Pad1) -> /TONE_P3
- C10 pad 2: Net-(C1-Pad1) -> Net-(C10-Pad2)
- C11 pad 1: Net-(C11-Pad1) -> /TONE_P1
- C11 pad 2: Net-(C11-Pad2) -> /GND
- C12 pad 2: Net-(C12-Pad2) -> /TONE_P2
- C13 pad 1: Net-(C12-Pad1) -> Net-(C13-Pad1)
- C13 pad 2: Net-(C13-Pad2) -> /VOL_P1
- C2 pad 2: /VOL_P1 -> Net-(C1-Pad1)
- C3 pad 1: Net-(C3-Pad1) -> /SUS_P3
- C3 pad 2: /TONE_P2 -> Net-(C2-Pad1)
- C4 pad 1: /SUS_P3 -> /SUS_P2
- C4 pad 2: Net-(C10-Pad1) -> Net-(C4-Pad2)
- C5 pad 1: /SUS_P2 -> Net-(C5-Pad1)
- C6 pad 2: Net-(C12-Pad2) -> Net-(C5-Pad2)
- C7 pad 1: Net-(C7-Pad1) -> Net-(C6-Pad1)
- C7 pad 2: Net-(C11-Pad2) -> Net-(C7-Pad2)
- C8 pad 1: /TONE_P1 -> Net-(C8-Pad1)
- C8 pad 2: /GND -> Net-(C8-Pad2)
- C9 pad 1: /TONE_P3 -> Net-(C10-Pad2)
- C9 pad 2: Net-(C11-Pad1) -> Net-(C8-Pad2)
- D1 pad 1: Net-(C7-Pad1) -> /+9V
- D1 pad 2: Net-(C11-Pad1) -> Net-(D1-Pad2)
- D2 pad 1: Net-(C11-Pad1) -> Net-(C6-Pad1)
- D2 pad 2: Net-(C7-Pad1) -> Net-(C5-Pad1)
- D3 pad 1: Net-(C6-Pad1) -> Net-(C5-Pad1)
- D3 pad 2: Net-(C12-Pad1) -> Net-(C6-Pad1)
- D4 pad 1: Net-(C12-Pad1) -> Net-(C10-Pad2)
- D4 pad 2: Net-(C6-Pad1) -> Net-(C8-Pad1)
- D5 pad 1: Net-(D5-Pad1) -> Net-(C8-Pad1)
- D5 pad 2: Net-(D5-Pad2) -> Net-(C10-Pad2)
- D6 pad 1: /+9V -> Net-(D6-Pad1)
- J1 pad 2: Net-(D6-Pad2) -> Net-(D1-Pad2)
- J3 pad 4: Net-(D5-Pad2) -> Net-(D6-Pad2)
- Q1 pad 1: Net-(C3-Pad1) -> Net-(C1-Pad1)
- Q2 pad 1: Net-(C11-Pad2) -> Net-(C5-Pad2)
- Q2 pad 3: Net-(C11-Pad1) -> Net-(C6-Pad1)
- Q3 pad 1: Net-(C12-Pad2) -> Net-(C8-Pad2)
- Q3 pad 3: Net-(C12-Pad1) -> Net-(C10-Pad2)
- Q4 pad 1: Net-(C1-Pad1) -> Net-(C12-Pad1)
- Q4 pad 3: Net-(C10-Pad1) -> Net-(C13-Pad1)
- R1 pad 1: Net-(D5-Pad1) -> Net-(C1-Pad2)
- R1 pad 2: Net-(J3-Pad2) -> Net-(R1-Pad2)
- R10 pad 1: Net-(Q2-Pad2) -> /+9V
- R10 pad 2: /GND -> Net-(C6-Pad1)
- R11 pad 1: /+9V -> Net-(Q2-Pad2)
- R11 pad 2: Net-(C11-Pad1) -> /GND
- R12 pad 1: Net-(C13-Pad2) -> Net-(C7-Pad2)
- R12 pad 2: Net-(C11-Pad2) -> Net-(C8-Pad2)
- R13 pad 1: Net-(C10-Pad1) -> Net-(C8-Pad2)
- R13 pad 2: /+9V -> /GND
- R14 pad 1: /GND -> Net-(C10-Pad2)
- R14 pad 2: Net-(C1-Pad1) -> Net-(C8-Pad2)
- R15 pad 1: Net-(C11-Pad1) -> /+9V
- R15 pad 2: Net-(C11-Pad2) -> Net-(C10-Pad2)
- R16 pad 1: Net-(C11-Pad2) -> Net-(Q3-Pad2)
- R17 pad 1: Net-(C12-Pad1) -> /TONE_P1
- R17 pad 2: Net-(C12-Pad2) -> Net-(C10-Pad2)
- R18 pad 1: /+9V -> /GND
- R18 pad 2: Net-(C12-Pad1) -> /TONE_P3
- R19 pad 1: Net-(C5-Pad2) -> /+9V
- R19 pad 2: Net-(C12-Pad2) -> Net-(C12-Pad1)
- R2 pad 1: Net-(C1-Pad2) -> /GND
- R2 pad 2: Net-(R2-Pad2) -> Net-(C1-Pad1)
- R20 pad 1: Net-(C12-Pad2) -> Net-(C12-Pad1)
- R21 pad 1: Net-(Q3-Pad2) -> /+9V
- R21 pad 2: /GND -> Net-(C13-Pad1)
- R22 pad 1: /GND -> Net-(Q4-Pad2)
- R22 pad 2: Net-(Q4-Pad2) -> /GND
- R23 pad 1: /SUS_P1 -> Net-(D6-Pad1)
- R23 pad 2: /GND -> Net-(J3-Pad2)
- R3 pad 1: Net-(C3-Pad1) -> Net-(C2-Pad1)
- R3 pad 2: /GND -> Net-(C1-Pad1)
- R4 pad 1: Net-(Q1-Pad2) -> Net-(C2-Pad1)
- R4 pad 2: /GND -> /+9V
- R5 pad 2: /TONE_P3 -> Net-(Q1-Pad2)
- R6 pad 1: /+9V -> /SUS_P1
- R6 pad 2: Net-(C2-Pad1) -> /GND
- R7 pad 1: /+9V -> Net-(C4-Pad2)
- R7 pad 2: Net-(C3-Pad1) -> Net-(C5-Pad2)
- R8 pad 1: /TONE_P1 -> Net-(C5-Pad2)
- R8 pad 2: Net-(C11-Pad1) -> /GND
- R9 pad 1: Net-(C10-Pad1) -> Net-(C6-Pad1)
- R9 pad 2: Net-(C1-Pad1) -> Net-(C5-Pad2)
- SW_EN1 pad 1: Net-(SW_EN1-Pad1) -> /VOL_P2
- SW_EN1 pad 3: /VOL_P2 -> Net-(SW_EN1-Pad3)
- SW_EN1 pad 7: Net-(SW_EN1-Pad1) -> Net-(R1-Pad2)
- SW_EN1 pad 9: Net-(R2-Pad2) -> Net-(SW_EN1-Pad3)
Routing:
- net /GND: track 85.4 -> 205.0 mm
- net /+9V: track 35.4 -> 114.1 mm, vias 0 -> 5
- net /VOL_P2: track 62.0 -> 0.00 mm
- net Net-(C12-Pad1): track 30.9 -> 81.7 mm, vias 0 -> 4
- net /SUS_P3: track 0.34 -> 49.3 mm
- net Net-(J_IN1-Pad1): track 4.38 -> 52.6 mm, vias 0 -> 2
- net /SUS_P2: track 0.00 -> 32.0 mm
- net Net-(J_IN1-Pad2): track 31.0 -> 0.00 mm
- net Net-(C5-Pad2): track 0.00 -> 29.7 mm
- net Net-(C6-Pad1): track 0.00 -> 26.5 mm
- net Net-(C11-Pad1): track 25.7 -> 0.00 mm
- net Net-(C3-Pad1): track 17.8 -> 0.00 mm
- net /SUS_P1: track 0.00 -> 17.4 mm
- net Net-(C11-Pad2): track 17.2 -> 0.00 mm
- net Net-(R1-Pad2): track 0.00 -> 15.9 mm, vias 0 -> 2
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
Commit message: update
Parts:
- moved TONE1 122.0 mm to (136.3, 123.8)
- moved VOLUME1 107.7 mm to (122.3, 123.7)
- moved SUSTAIN1 95.6 mm to (150.4, 123.7)
- moved R20 51.7 mm to (58.1, 168.3), turned to 180 degrees
- moved D6 40.2 mm to (149.3, 132.0), turned to 270 degrees
- moved R13 37.3 mm to (83.8, 130.8)
- moved C7 35.7 mm to (92.5, 146.2), turned to 90 degrees
- moved R18 34.7 mm to (71.6, 154.4), turned to 180 degrees
- moved C6 32.4 mm to (91.3, 149.1), turned to 180 degrees
- moved R23 28.5 mm to (140.6, 131.9), turned to 270 degrees
- moved R16 25.8 mm to (92.9, 134.4), turned to 270 degrees
- moved J3 25.4 mm to (135.7, 131.9), turned to 270 degrees
- moved R21 22.8 mm to (69.1, 119.9)
- moved R12 20.9 mm to (91.4, 143.1), turned to 180 degrees
- moved C10 19.8 mm to (64.5, 146.6), turned to 0 degrees
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Routing:
- net /GND: track 205.0 -> 348.0 mm, vias 2 -> 8
- net /VOL_P2: track 0.00 -> 91.2 mm
- net /LED_AN: track 9.10 -> 87.7 mm, vias 0 -> 2
- net Net-(C13-Pad1): track 0.18 -> 74.0 mm
- net Net-(C10-Pad2): track 0.00 -> 68.1 mm, vias 0 -> 4
- net Net-(J3-Pad11): track 0.00 -> 61.8 mm
- net Net-(J3-Pad9): track 0.00 -> 47.5 mm
- net Net-(J3-Pad7): track 0.00 -> 32.4 mm
- net Net-(J3-Pad8): track 0.00 -> 30.3 mm
- net Net-(C8-Pad2): track 0.00 -> 27.2 mm
- net Net-(J3-Pad10): track 0.00 -> 24.4 mm
- net /TONE_P3: track 0.00 -> 23.7 mm, vias 0 -> 4
- net /+9V: track 114.1 -> 136.3 mm
- net Net-(D6-Pad2): track 0.00 -> 20.3 mm
- net Net-(C8-Pad1): track 0.00 -> 14.9 mm, vias 0 -> 2
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Other:
- board size 155.2 x 217.4 mm -> 214.3 x 217.4 mm
