File: BMP_BasicClone/BMP_BasicClone.kicad_pcb (KiCad board)
At the start: 2 copper layers, 214.3 x 217.4 mm, 55 parts, among them J1 BARREL_JACK, J2 CONN_02X06, J3 CONN_02X06, Q1 MMBT3904, Q2 MMBT3904, Q3 MMBT3904, Q4 MMBT3904

Commit message: Update
Parts:
- removed J2, J3: CONN_02X06, Pin_Headers:Pin_Header_Straight_2x06_Pitch2.54mm
- added J_AUX2MAIN_1: CONN_01X06, Pin_Headers:Pin_Header_Straight_1x06_Pitch2.54mm, F.Cu at (153.2, 131.8)
- added J_AUX2MAIN_2: CONN_01X06, Pin_Headers:Pin_Header_Straight_1x06_Pitch2.54mm, F.Cu at (114.4, 132.2)
- added J_MAIN2AUX_1: CONN_01X06, Pin_Headers:Pin_Header_Straight_1x06_Pitch2.54mm, F.Cu at (94.2, 133.1)
- added J_MAIN2AUX_2: CONN_01X06, Pin_Headers:Pin_Header_Straight_1x06_Pitch2.54mm, F.Cu at (56.0, 133.5)
- C1, C10, C11, C12, C13, C2, C3, C4, C5, C6, C7, C8, C9, D1, D2, D3, D4, D5, Q1, Q2, Q3, Q4, R1, R10, R11, R12, R13, R14, R15, R16, R17, R18, R19, R2, R20, R21, R22, R23, R3, R4, R5, R6, R7, R8, R9: moved to B.Cu
- moved R19 49.5 mm to (58.0, 166.2)
- moved R21 36.7 mm to (58.0, 154.9), turned to 180 degrees
- moved C13 32.2 mm to (56.3, 152.5), turned to 0 degrees
- moved C12 30.5 mm to (57.9, 168.8), turned to 0 degrees
- moved R16 27.1 mm to (69.0, 121.7), turned to 180 degrees
- moved C8 26.7 mm to (64.0, 125.6)
- moved R17 23.1 mm to (77.9, 123.7), turned to 90 degrees
- moved R18 22.3 mm to (76.2, 132.6), turned to 0 degrees
- moved C10 21.2 mm to (77.5, 129.8), turned to 180 degrees
- moved D6 20.9 mm to (133.9, 117.9)
- moved C11 20.3 mm to (80.5, 123.7), turned to 90 degrees
- moved Q3 19.6 mm to (73.8, 122.8), turned to 0 degrees
- moved D5 19.6 mm to (74.0, 117.6)
- moved R14 18.6 mm to (68.6, 132.8), turned to 180 degrees
- moved R20 18.3 mm to (59.7, 186.6), turned to 270 degrees
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Routing:
- net /GND: track 348.0 -> 262.2 mm, vias 8 -> 10
- net Net-(C12-Pad1): track 88.3 -> 22.8 mm, vias 2 -> 0
- net /TONE_P2: track 3.62 -> 68.8 mm, vias 0 -> 4
- net Net-(C13-Pad1): track 74.0 -> 31.1 mm
- net Net-(J_AUX2MAIN_1-Pad6): track 61.8 -> 20.5 mm
- net Net-(J_AUX2MAIN_1-Pad5): track 47.5 -> 11.3 mm
- net /VOL_P2: track 91.2 -> 60.6 mm
- net Net-(C10-Pad2): track 68.1 -> 38.2 mm, vias 4 -> 0
- net Net-(J_AUX2MAIN_1-Pad4): track 32.4 -> 6.95 mm
- net Net-(J_AUX2MAIN_2-Pad3): track 30.3 -> 6.67 mm
- net Net-(C8-Pad2): track 27.2 -> 47.0 mm, vias 0 -> 2
- net Net-(J_AUX2MAIN_1-Pad3): track 8.45 -> 26.0 mm
- net Net-(J_AUX2MAIN_2-Pad6): track 5.70 -> 20.9 mm
- net /VOL_P1: track 5.51 -> 19.6 mm
- net Net-(J_AUX2MAIN_2-Pad2): track 24.4 -> 10.6 mm
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Other:
- outline, holes or cut-outs redrawn

Commit message: Update
Parts:
- moved R23 59.0 mm to (120.7, 172.8)
- moved J_AUX2MAIN_1 58.6 mm to (142.5, 189.5)
- moved SUSTAIN1 58.3 mm to (136.7, 183.3)
- moved D6 58.3 mm to (123.2, 175.2)
- moved TONE1 58.3 mm to (125.9, 192.1)
- moved VOLUME1 58.3 mm to (115.1, 183.6)
- moved J_AUX2MAIN_2 58.2 mm to (104.3, 189.5)
- moved C7 2.08 mm to (86.9, 149.0), turned to 90 degrees
- moved R12 1.18 mm to (84.3, 147.1), turned to 90 degrees
- moved SW_EN1 0.46 mm to (75.1, 186.9)
- moved J_MAIN2AUX_2 0.38 mm to (56.0, 133.1)
- moved J_MAIN2AUX_1 0.13 mm to (94.1, 133.1)
Routing:
- net Net-(C10-Pad2): track 38.2 -> 31.4 mm
- net /GND: track 262.2 -> 265.4 mm
- net Net-(J_AUX2MAIN_2-Pad6): track 20.9 -> 18.4 mm
- net Net-(C8-Pad1): track 15.9 -> 18.1 mm
- net Net-(C7-Pad2): track 4.58 -> 2.75 mm
- net Net-(C1-Pad1): track 13.7 -> 15.1 mm
- net Net-(J_IN1-Pad1): track 61.2 -> 62.2 mm
- net Net-(D6-Pad1): track 2.83 -> 3.76 mm
- net Net-(C12-Pad1): track 22.8 -> 23.6 mm
- net /LED_AN: track 82.3 -> 81.7 mm
- net Net-(SW_EN1-Pad3): track 15.4 -> 14.8 mm
- net /+9V: track 142.9 -> 142.3 mm
- net /TONE_P3: track 20.3 -> 20.8 mm
- net Net-(D6-Pad2): track 20.3 -> 19.7 mm
- net Net-(J_AUX2MAIN_2-Pad3): track 6.67 -> 6.14 mm
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Other:
- board size 214.3 x 217.4 mm -> 90.3 x 91.9 mm
- rule trace_min: 0.2 -> 0.1524

Commit message: Updates
Parts:
- C1, C10, C11, C12, C13, C2, C3, C4, C5, C6, C7, C8, C9: footprint Capacitors_SMD:C_0805 -> Capacitors_SMD:C_0805_HandSoldering
- D1, D2, D3, D4, D5: footprint Diodes_SMD:D_SOD-523 -> Diodes_SMD:D_SOD-323
- R1, R10, R11, R12, R13, R14, R15, R16, R17, R18, R19, R2, R20, R21, R22, R23, R3, R4, R5, R6, R7, R8, R9: footprint Resistors_SMD:R_0805 -> Resistors_SMD:R_0805_HandSoldering
- moved D6 54.8 mm to (74.9, 201.1)
- moved VOLUME1 54.8 mm to (66.8, 209.5)
- moved J_AUX2MAIN_1 54.8 mm to (94.2, 215.4)
- moved TONE1 54.8 mm to (77.6, 218.0)
- moved J_AUX2MAIN_2 54.8 mm to (56.0, 215.4)
- moved R23 54.8 mm to (72.5, 198.8)
- moved SUSTAIN1 54.8 mm to (88.4, 209.2)
- moved C4 16.0 mm to (92.2, 145.0)
- moved R7 15.8 mm to (92.2, 149.9)
- moved R2 6.12 mm to (86.1, 175.2), turned to 0 degrees
- moved R20 5.31 mm to (62.9, 182.3), turned to 0 degrees
- moved C1 5.08 mm to (88.7, 179.1), turned to 270 degrees
- moved C5 4.38 mm to (90.6, 160.6)
- moved R22 3.55 mm to (59.4, 185.8), turned to 0 degrees
- moved R8 2.93 mm to (89.6, 147.6), turned to 90 degrees
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Connections:
- SW_EN1 pad 4: Net-(SW_EN1-Pad4) -> /LED_AN
- SW_EN1 pad 6: /LED_AN -> Net-(SW_EN1-Pad6)
Routing:
- net /GND: track 265.4 -> 245.8 mm
- net /SUS_P2: track 46.2 -> 30.1 mm
- net Net-(C6-Pad1): track 32.0 -> 39.2 mm
- net /LED_AN: track 81.7 -> 75.2 mm
- net Net-(C5-Pad1): track 7.18 -> 13.1 mm
- net /+9V: track 142.3 -> 137.7 mm
- net Net-(C10-Pad2): track 31.4 -> 34.7 mm
- net /VOL_P1: track 20.0 -> 16.7 mm
- net Net-(J_IN1-Pad1): track 62.2 -> 65.5 mm
- net Net-(C7-Pad2): track 2.75 -> 5.02 mm
- net /TONE_P1: track 19.3 -> 21.5 mm
- net /TONE_P3: track 20.8 -> 19.0 mm
- net Net-(Q4-Pad2): track 3.42 -> 5.18 mm
- net Net-(C13-Pad1): track 30.8 -> 32.5 mm
- net Net-(C8-Pad2): track 46.9 -> 45.4 mm
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Other:
- board size 90.3 x 91.9 mm -> 42.1 x 116 mm
- rule trace_min: 0.1524 -> 0.0254
